File: Hardware/Bongo-Cat-Fidget-Toy/_autosave-Bongo-Cat-Fidget-Toy.kicad_pcb (KiCad board)
At the start: 2 copper layers, 42.5 x 47 mm, 40 parts, among them J1 Conn_01x30, J2 Conn_01x04, J3 Conn_01x04, SW1 SW_Push, SW2 SW_Push, SW3 SW_MEC_5E, SW5 SW_SPDT_321, U1 STM32G030K8Tx, U2 MT3608, Y1 Crystal_GND24_Small

Commit message: Production version
Parts:
- moved L1 0.81 mm to (93.1, 50.9)
Changed lines of the file:
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@@
 	(footprint "Inductor_SMD:L_Changjiang_FNR5040S"
 		(layer "B.Cu")
-		(at 93.92 50.91 90)
+		(at 93.11 50.87 90)
 		(descr "Inductor, Changjiang, FNR5040S, 5.0x5.0x4.0mm, https://datasheet.lcsc.com/lcsc/1806131217_cjiang-Changjiang-Microelectronics-Tech-FNR5040S3R3NT_C167960.pdf")
 		(tags "Inductor wirewound power shielded")
