File: Hardware/Bongo-Cat-Fidget-Toy-Lite/Bongo-Cat-Fidget-Toy-Lite/Bongo-Cat-Fidget-Toy-Lite.kicad_sch (KiCad schematic)
At the start: 25 parts, among them J1 LYA130BG30-128064, J2 Conn_01x04, SW1 SW_Push, SW2 SW_Push, SW5 SW_SPDT_321, U101 TPS63802DLAR, U2 PY32F003F1xU

Commit message: Updated code and PCB
Connections:
- net PA2 is gone; now on net SDA: U2.18 (PA2)
- net PA3 is gone; now on net SCL: U2.19 (PA3)
- net SCL: no longer U2.10 (PB6)
- net SDA: no longer U2.11 (PB7)
- no-connect marks 12 -> 14

Commit message: Minor change
Parts:
- U2: LCSC (none) -> C3018714
Other:
- note added: "maybe change to PY32F030F28P6TU"
- note removed: "- Has internal pullup"
Changed lines of the file:
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@@
 		)
 	)
-	(text "- Has internal pullup"
+	(text "maybe change to PY32F030F28P6TU"
 		(exclude_from_sim no)
-		(at 60.452 178.308 0)
+		(at 66.548 177.8 0)
 		(effects
 			(font
@@
 			(at 78.74 140.97 0)
 			(hide yes)
+			(show_name no)
+			(do_not_autoplace no)
+			(effects
+				(font
+					(size 1.27 1.27)
+				)
+			)
+		)
+		(property "LCSC" "C3018714"
+			(at 78.74 140.97 0)
+			(hide yes)

Commit message: Lite PCB changes
Parts:
- removed J2: Conn_01x04, Connector_PinHeader_2.54mm:PinHeader_1x04_P2.54mm_Horizontal, symbol Connector_Generic:Conn_01x04
- added FID1, FID2, FID3: Fiducial, Fiducial:Fiducial_0.5mm_Mask1.5mm, symbol Mechanical:Fiducial
- added J4: Conn_ARM_SWD_TagConnect_TC2030-NL, Connector:Tag-Connect_TC2030-IDC-NL_2x03_P1.27mm_Vertical, symbol Connector:Conn_ARM_SWD_TagConnect_TC2030-NL
Connections:
- net 3V3: now also J4.1 (VCC)
- net GND: now also J4.5 (GND)
- net RST: now also J4.3 (~{RESET})
- net SWCLK: now also J4.4 (SWCLK)
- net SWDIO: now also J4.2 (SWDIO)
- no-connect marks 14 -> 15
